Commit message: gazebo testing

File: description/oculusprime.urdf (robot description, URDF)
Before this commit: robot oculusPrime, 1 links, 0 joints
Links:
- added link front_left_wheel_link, mass 0.05; collision cylinder length=0.046 radius=0.057; visual cylinder length=0.046 radius=0.057
- added link front_right_wheel_link, mass 0.05; collision cylinder length=0.046 radius=0.057; visual cylinder length=0.046 radius=0.057
- added link rear_left_wheel_link, mass 0.05; collision cylinder length=0.046 radius=0.057; visual cylinder length=0.046 radius=0.057
- added link rear_right_wheel_link, mass 0.05; collision cylinder length=0.046 radius=0.057; visual cylinder length=0.046 radius=0.057
- link base_link: geometry collision box size=.275 .19 .275; visual mesh filename=package://oculusprime/description/meshes/chassis.dae
Joints:
- added joint front_left_wheel_joint: type continuous, parent base_link, child front_left_wheel_link, origin xyz=0.0635 0.1186 0.057 rpy=0 1.5707 1.5707, axis 0 0 1
- added joint front_right_wheel_joint: type continuous, parent base_link, child front_right_wheel_link, origin xyz=0.0635 -0.1186 0.057 rpy=0 1.5707 1.5707, axis 0 0 1
- added joint rear_left_wheel_joint: type continuous, parent base_link, child rear_left_wheel_link, origin xyz=-0.0635 0.1186 0.057 rpy=0 1.5707 1.5707, axis 0 0 1
- added joint rear_right_wheel_joint: type continuous, parent base_link, child rear_right_wheel_link, origin xyz=-0.0635 -0.1186 0.057 rpy=0 1.5707 1.5707, axis 0 0 1
