Commit message: gazebo urdfs and launch

File: description/oculusprime.urdf.xacro (robot description, xacro)
@@ -1,4 +1,4 @@
 <?xml version='1.0'?>
-<robot name="oculus_prime">
+<robot name="oculusprime" xmlns:xacro="http://ros.org/wiki/xacro">
 	<link name="base_link">
 		<inertial>
@@ -149,4 +149,7 @@
 		</inertial>
 	</link>
+	<!-- astra -->
+	<xacro:include filename="$(find oculusprime)/description/astra.urdf.xacro"/>
+	<sensor_astra parent="base_link"/>
 	<!-- gazebo specific stuff -->
 	<gazebo reference="front_right_wheel_link">
@@ -205,8 +208,11 @@
 	      </imu>
       </sensor>
-	  </gazebo>
+	</gazebo>
 	<gazebo>
 		<plugin name="skidsteer_controller" filename="libgazebo_ros_skid_steer_drive.so">
-			<publish_tf>1</publish_tf>
+			<commandTopic>cmd_vel</commandTopic>
+			<broadcastTF>true</broadcastTF>
+			<odometryTopic>odom</odometryTopic>
+			<odometryFrame>odom</odometryFrame>
 			<leftFrontJoint>front_left_wheel_joint</leftFrontJoint>
 			<rightFrontJoint>front_right_wheel_joint</rightFrontJoint>
@@ -217,5 +223,10 @@
 			<torque>1.0</torque>
 			<robotBaseFrame>base_link</robotBaseFrame>
+			<updateRate>30</updateRate>
 		</plugin>
 	</gazebo>
+	<gazebo>
+		<plugin name="gazebo_joint_state_publisher" filename="libgazebo_ros_joint_state_publisher.so">
+		</plugin>
+	</gazebo>
 </robot>

File: description/oculusprime_simple.urdf (robot description, URDF)
Before this commit: robot oculusPrime, 1 links, 0 joints
Links:
- link base_link: geometry collision box size=0.275 0.283 0.306; visual mesh filename=package://oculusprime/description/meshes/oculus_prime_urdf.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 scale=0.0254 0.0254 0.0254
