Commit message: urdf details, imu noise

File: description/astra.urdf.xacro (robot description, xacro)
@@ -2,11 +2,11 @@
 <robot name="sensor_astra" xmlns:xacro="http://ros.org/wiki/xacro">
 	<!-- Xacro properties -->
-	<xacro:property name="astra_cam_py" value="-0.0125"/>
+	<xacro:property name="astra_cam_py" value="0.0125"/> <!-- -0.0125 -->
 	<xacro:property name="astra_depth_rel_rgb_py" value="0.0250" />
 	<xacro:property name="astra_cam_rel_rgb_py"   value="-0.0125" />
 	<xacro:property name="astra_dae_display_scale"   value="1" />
-	<xacro:property name="cam_px" value="-0.054" /> <!-- -0.087 -->
+	<xacro:property name="cam_px" value="-0.0545" /> <!-- -0.087 -->
 	<!--	<xacro:property name="cam_py" value="-0.0125" /> Y varies for different configurations. get sets in sensors_urdf -->
-	<xacro:property name="cam_pz" value="0.2870" />
+	<xacro:property name="cam_pz" value="0.2930" />
 	<xacro:property name="cam_or" value="0" />
 	<xacro:property name="cam_op" value="0" />
@@ -40,10 +40,8 @@
     <link name="camera_link">
       <visual>
-<!--
-        <origin xyz="-0.04 0.02 -0.01" rpy="0 0 0"/>
--->
-        <origin xyz="0 0 0" rpy="0 0 0"/>
+        <origin xyz="-.030 0 -.008" rpy="0 0 0"/>
         <geometry>
-          <mesh filename="package://oculusprime/description/meshes/orbbec_astra_camera.dae" scale="${astra_dae_display_scale} ${astra_dae_display_scale} ${astra_dae_display_scale}"/>
+          <mesh filename="package://oculusprime/description/meshes/orbbec_astra_camera.dae"
+			scale="${astra_dae_display_scale} ${astra_dae_display_scale} ${astra_dae_display_scale}"/>
         </geometry>
       </visual>

File: description/oculusprime.urdf.xacro (robot description, xacro)
@@ -1,7 +1,8 @@
 <?xml version='1.0'?>
 <robot name="oculusprime" xmlns:xacro="http://ros.org/wiki/xacro">
+<xacro:property name="M_PI" value="3.1415926535897931" />
 	<link name="base_link">
 		<inertial>
-			<origin xyz="0 0 0.08" rpy="0 0 0" />
+			<origin xyz="0 0 0.06" rpy="0 0 0" />
 			<mass value="4.0"/>
 			<inertia ixx="0.0227"
@@ -13,22 +14,22 @@
 		</inertial>
 		<collision>
-			<origin xyz="0 0 0.155" rpy="0 0 0" />
-			<geometry>
-				<box size=".275 .19 .275"/>
-			</geometry>
-		</collision>
-		<visual>
-			<origin xyz="0 0 0" rpy="0 0 0" />
+			<origin xyz="-0.0064 0 0.1517" rpy="0 0 0" />
+			<geometry>
+				<box size=".2818 .19 .2595"/>
+			</geometry>
+		</collision>
+		<visual>
+			<origin xyz="0.0127 0 .0808" rpy="0 0 ${M_PI/2}" />
 			<geometry>
 				<mesh filename="package://oculusprime/description/meshes/chassis.dae" />
 			</geometry>
-			<material name="grey">
-			<color rgba="0.4 0.4 0.4 1.0"/>
-			</material>
-		</visual>
-	</link>
+		</visual>
+	</link>
+	<material name="black">
+		<color rgba="0.1 0.1 0.1 1.0"/>
+	</material>
 	<!-- wheels -->
 	<joint type="continuous" name="front_right_wheel_joint">
-		<origin xyz="0.0635 -0.1186 0.057" rpy="0 1.5707 1.5707"/>
+		<origin xyz="0.0635 -0.1186 0.057" rpy="0 ${M_PI/2} ${M_PI/2}"/>
 		<parent link="base_link"/>
 		<child link="front_right_wheel_link"/>
@@ -47,7 +48,5 @@
 				<cylinder radius="0.057" length="0.046" />
 			</geometry>
-			<material name="black">
-				<color rgba="0.05 0.05 0.05 1.0"/>
-			</material>
+			<material name="black"/>
 		</visual>
 		<inertial>
@@ -60,5 +59,5 @@
 	</link>
 	<joint type="continuous" name="front_left_wheel_joint">
-		<origin xyz="0.0635 0.1186 0.057" rpy="0 1.5707 1.5707"/>
+		<origin xyz="0.0635 0.1186 0.057" rpy="0 ${M_PI/2} ${M_PI/2}"/>
 		<child link="front_left_wheel_link"/>
 		<parent link="base_link"/>
@@ -77,7 +76,5 @@
 				<cylinder radius="0.057" length="0.046" />
 			</geometry>
-			<material name="black">
-				<color rgba="0.05 0.05 0.05 1.0"/>
-			</material>
+			<material name="black"/>
 		</visual>
 		<inertial>
@@ -90,5 +87,5 @@
 	</link>
 	<joint type="continuous" name="rear_right_wheel_joint">
-		<origin xyz="-0.0635 -0.1186 0.057" rpy="0 1.5707 1.5707"/>
+		<origin xyz="-0.0635 -0.1186 0.057" rpy="0 ${M_PI/2} ${M_PI/2}"/>
 		<child link="rear_right_wheel_link"/>
 		<parent link="base_link"/>
@@ -107,7 +104,5 @@
 				<cylinder radius="0.057" length="0.046" />
 			</geometry>
-			<material name="black">
-				<color rgba="0.05 0.05 0.05 1.0"/>
-			</material>
+			<material name="black"/>
 		</visual>
 		<inertial>
@@ -120,5 +115,5 @@
 	</link>
 	<joint type="continuous" name="rear_left_wheel_joint">
-		<origin xyz="-0.0635 0.1186 0.057" rpy="0 1.5707 1.5707"/>
+		<origin xyz="-0.0635 0.1186 0.057" rpy="0 ${M_PI/2} ${M_PI/2}"/>
 		<child link="rear_left_wheel_link"/>
 		<parent link="base_link"/>
@@ -137,7 +132,5 @@
 				<cylinder radius="0.057" length="0.046" />
 			</geometry>
-			<material name="black">
-				<color rgba="0.05 0.05 0.05 1.0"/>
-			</material>
+			<material name="black"/>
 		</visual>
 		<inertial>
@@ -160,4 +153,5 @@
 		<minDepth>0.001</minDepth>
 		<maxVel>1.0</maxVel>
+		<material>Gazebo/DarkGrey</material>
 	</gazebo>
 	<gazebo reference="front_left_wheel_link">
@@ -168,4 +162,5 @@
 		<minDepth>0.001</minDepth>
 		<maxVel>1.0</maxVel>
+		<material>Gazebo/DarkGrey</material>
 	</gazebo>
 	<gazebo reference="rear_right_wheel_link">
@@ -176,4 +171,5 @@
 		<minDepth>0.001</minDepth>
 		<maxVel>1.0</maxVel>
+		<material>Gazebo/DarkGrey</material>
 	</gazebo>
 	<gazebo reference="rear_left_wheel_link">
@@ -184,5 +180,21 @@
 		<minDepth>0.001</minDepth>
 		<maxVel>1.0</maxVel>
-	</gazebo>
+		<material>Gazebo/DarkGrey</material>
+	</gazebo>
+	<joint name="gyro_joint" type="fixed">
+      <axis xyz="0 1 0"/>
+      <origin xyz="0 0 0" rpy="0 0 0"/>
+      <parent link="base_link"/>
+      <child link="gyro_link"/>
+    </joint>
+    <link name="gyro_link">
+      <inertial>
+        <mass value="0.001"/>
+        <origin xyz="0 0 0" rpy="0 0 0"/>
+        <inertia ixx="0.0001" ixy="0" ixz="0"
+                 iyy="0.000001" iyz="0"
+                 izz="0.0001"/>
+      </inertial>
+    </link>
 	<gazebo reference="gyro_link">
 	   <sensor type="imu" name="imu">
